Commit message: change absolute path to relative, fix 'fixed frame' in rviz.

File: youbot_description/robots/youbot_arm.urdf.xacro (robot description, xacro)
@@ -12,5 +12,5 @@
   <!-- youbot arm -->
   <xacro:include filename="$(find youbot_description)/urdf/youbot_arm/arm.urdf.xacro" />
-  <!-- youbot arm -->
+  <!-- youbot gripper -->
   <xacro:include filename="$(find youbot_description)/urdf/youbot_gripper/gripper.urdf.xacro" />
   <!-- generic simulator_gazebo plugins for starting mechanism control, ros time, ros battery -->
@@ -39,5 +39,5 @@
   </xacro:youbot_arm>
   <xacro:youbot_gripper name="gripper" parent="arm_link_5">
-    <origin xyz="0 0 0" rpy="0 0 0" />
+    <origin xyz="0 0 0" rpy="0 ${-M_PI/2} ${M_PI}" />
   </xacro:youbot_gripper>
 </robot>
